File: rp2040-bakeneko65.kicad_pcb (KiCad board)
At the start: 2 copper layers, 180 parts, among them J1 SM04B-SRSS-TB, SW1 1u, SW10 1u, SW11 1u, SW12 1u, SW13 1u, SW14 1u, SW15 1u, SW16 1u, SW17 2u, SW18 1.5u, SW19 1u, SW2 1u, SW20 1u, SW21 1u, SW22 1u, SW23 1u, SW24 1u, SW25 1u, SW26 1u, SW27 1u, SW28 1u, SW29 1u, SW3 1u, SW30 1u, SW31 1.5u, SW32 ISO Enter, SW33 1u, SW34 1.25u, SW35 1.75u, SW36 1u, SW37 1u, SW38 1u, SW39 1u, SW4 1u, SW40 1u, SW41 1u, SW42 1u, SW43 1u, SW44 1u, SW45 1u, SW46 1u, SW47 2.25u, SW48 1u, SW49 1u, SW5 1u, SW50 2.25u, SW51 1.25u, SW52 1u, SW53 1u, SW54 1u, SW55 1u, SW56 1u, SW57 1u, SW58 1u, SW59 1u, SW6 1u, SW60 1u, SW61 1u, SW62 1u, SW63 1u, SW64 1u, SW65 1u, SW66 1.5u, SW67 1u, SW68 1.5u, SW69 7u, SW7 1u, SW70 1.25u, SW71 1.5u, SW72 1u, SW73 1u, SW74 1u, SW75 1.25u, SW76 1.25u, SW77 1.25u, SW78 6.25u, SW79 1.25u, SW8 1u, SW80 SW_Push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

Commit message: Add outline
Parts:
- moved C11 86.2 mm to (452.3, 123.8)
- moved C14 86.2 mm to (468.0, 111.5)
- moved C15 86.2 mm to (453.8, 120.8)
- moved C16 86.2 mm to (458.2, 120.5)
- moved C2 86.2 mm to (452.3, 126.8)
- moved C6 86.2 mm to (447.9, 125.2)
- moved C7 86.2 mm to (456.8, 123.8)
- moved C8 86.2 mm to (449.4, 120.8)
- moved C9 86.2 mm to (447.9, 128.2)
- moved D15 86.2 mm to (521.5, 102.3)
- moved D20 86.2 mm to (527.2, 102.3)
- moved D27 86.2 mm to (533.0, 102.3)
- moved D29 86.2 mm to (515.7, 102.3)
- moved D31 86.2 mm to (544.5, 102.3)
- moved D47 86.2 mm to (556.0, 102.3)
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Other:
- board outline added: 303.8 x 94.2 mm

Commit message: A couple switches
Parts:
- C1, C10, C11, C12, C13, C14, C15, C16, C17, C2, C3, C4, C5, C6, C7, C8, C9, D1, D10, D11, D12, D13, D14, D15, D16, D17, D18, D19, D2, D20, D21, D22, D23, D24, D25, D26, D27, D28, D29, D3, D30, D31, D32, D33, D34, D35, D36, D37, D38, D39, D4, D40, D41, D42, D43, D44, D45, D46, D47, D48, D49, D5, D50, D51, D52, D53, D54, D55, D56, D57, D58, D59, D6, D60, D61, D62, D63, D64, D65, D66, D67, D68, D69, D7, D70, D71, D8, D9, J1, R1, R2, R3, R4, SW80, U1, U2, U3, Y1: moved to B.Cu
- moved SW63 382.2 mm to (89.7, 96.5)
- moved SW34 374.7 mm to (70.6, 96.5)
- moved D22 273.1 mm to (451.9, 165.3), turned to 180 degrees
- moved D4 265.4 mm to (457.7, 165.3), turned to 180 degrees
- moved D26 258.0 mm to (463.4, 165.3), turned to 180 degrees
- moved D59 250.9 mm to (469.2, 165.3), turned to 180 degrees
- moved D66 244.2 mm to (474.9, 165.3), turned to 180 degrees
- moved D10 235.1 mm to (453.2, 121.1), turned to 180 degrees
- moved D3 235.1 mm to (453.2, 124.5), turned to 180 degrees
- moved D23 226.4 mm to (458.9, 124.5), turned to 180 degrees
- moved D5 226.4 mm to (458.9, 131.2), turned to 180 degrees
- moved D65 226.4 mm to (458.9, 127.8), turned to 180 degrees
- moved D9 226.4 mm to (458.9, 121.1), turned to 180 degrees
- moved D64 222.3 mm to (484.6, 161.2), turned to 180 degrees
- moved D16 218.1 mm to (464.7, 127.8), turned to 180 degrees
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Other:
- outline, holes or cut-outs redrawn

Commit message: Some more switches
Parts:
- moved SW1 522.3 mm to (53.1, 100.6)
- moved SW3 495.9 mm to (91.2, 100.6)
- moved SW5 492.3 mm to (129.3, 100.6)
- moved SW4 439.7 mm to (110.2, 100.6)
- moved SW7 433.2 mm to (167.4, 100.6)
- moved SW63 412.1 mm to (482.1, -29.2)
- moved SW34 400.0 mm to (442.7, -50.3)
- moved SW2 386.5 mm to (72.1, 100.6)
- moved SW13 366.5 mm to (281.7, 100.6)
- moved SW10 360.3 mm to (224.5, 100.6)
- moved SW6 348.7 mm to (148.3, 100.6)
- moved SW8 342.5 mm to (186.4, 100.6)
- moved SW12 328.1 mm to (262.6, 100.6)
- moved SW15 317.4 mm to (319.8, 100.6)
- moved SW11 303.9 mm to (243.6, 100.6)
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Other:
- outline, holes or cut-outs redrawn

Commit message: Move switches a bit
Parts:
- moved SW13 0.24 mm to (281.8, 100.8)
- moved SW14 0.24 mm to (300.8, 100.8)
- moved SW15 0.24 mm to (319.9, 100.8)
- moved SW9 0.24 mm to (205.6, 100.8)
- moved SW2 0.24 mm to (72.2, 100.8)
- moved SW1 0.24 mm to (53.2, 100.8)
- moved SW10 0.24 mm to (224.6, 100.8)
- moved SW11 0.24 mm to (243.7, 100.8)
- moved SW3 0.24 mm to (91.3, 100.8)
- moved SW4 0.24 mm to (110.3, 100.8)
- moved SW5 0.24 mm to (129.4, 100.8)
- moved SW6 0.24 mm to (148.4, 100.8)
- moved SW7 0.24 mm to (167.5, 100.8)
- moved SW8 0.24 mm to (186.5, 100.8)
- moved SW12 0.24 mm to (262.7, 100.8)
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Other:
- outline, holes or cut-outs redrawn

Commit message: Even more switches
Parts:
- moved SW18 561.7 mm to (57.1, 119.1)
- moved SW35 506.1 mm to (59.5, 138.1)
- moved SW41 486.3 mm to (181.0, 138.1)
- moved SW21 482.2 mm to (119.1, 119.1)
- moved SW22 469.9 mm to (138.1, 119.1)
- moved SW43 457.3 mm to (219.1, 138.1)
- moved SW40 450.5 mm to (161.9, 138.1)
- moved SW24 441.3 mm to (176.2, 119.1)
- moved SW34 431.4 mm to (54.6, 138.1)
- moved SW36 412.8 mm to (85.7, 138.1)
- moved SW27 411.4 mm to (233.4, 119.1)
- moved SW37 407.7 mm to (104.8, 138.1)
- moved SW19 407.6 mm to (81.0, 119.1)
- moved SW44 381.3 mm to (238.1, 138.1)
- moved SW25 364.7 mm to (195.3, 119.1)
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Other:
- outline, holes or cut-outs redrawn

Commit message: Correct stabs
Parts:
- added S1: Back, marbastlib-mx:STAB_MX_2u, F.Cu at (383.4, -85.7)
- added S2: LShift, marbastlib-mx:STAB_MX_2u, F.Cu at (263.2, -85.7)
- added S3: ISO Enter, marbastlib-mx:STAB_MX_2u, F.Cu at (263.2, -44.1)
- added S4: 7u Space, marbastlib-mx:STAB_MX_P_7u, F.Cu at (263.2, -64.9)
- added S5: 6.25u Space, marbastlib-mx:STAB_MX_P_6.25u, F.Cu at (383.4, -106.6)
- added S6: Left Split Space, marbastlib-mx:STAB_MX_P_2u, F.Cu at (263.2, -23.2)
- added S7: Right Split Space, marbastlib-mx:STAB_MX_P_2u, F.Cu at (263.2, -106.6)
- C1: footprint Capacitor_SMD:C_0805_2012Metric -> marbastlib-mx:STAB_MX_2u
- SW63: value 1u -> 1.75u

Commit message: oops, forgot ANSI enter
Parts:
- added S8: Enter, marbastlib-mx:STAB_MX_2u, F.Cu at (261.9, -126.2)
- moved S6 2.60 mm to (263.2, -20.6)
- moved S4 1.40 mm to (261.9, -64.3)
- moved S2 1.26 mm to (261.9, -85.7)
- moved S7 1.26 mm to (261.9, -106.6)
- moved S3 1.20 mm to (263.2, -42.9)
Changed lines of the file:
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@@
   )
   (footprint "marbastlib-mx:STAB_MX_2u" (layer "F.Cu")
-    (at 263.20125 -85.725)
+    (at 261.9375 -85.725)
     (descr "Footprint for Cherry Clip/Screw in type stabilizers, 2u")
     (property "Sheetfile" "SwitchMatrix.kicad_sch")
@@
   )
   (footprint "marbastlib-mx:STAB_MX_P_2u" (layer "F.Cu")
-    (at 263.20125 -106.555)
+    (at 261.9375 -106.555)
     (descr "Footprint for Cherry Clip/Screw in type stabilizers, 2u")
     (property "Sheetfile" "SwitchMatrix.kicad_sch")
@@
   )
   (footprint "marbastlib-mx:STAB_MX_P_2u" (layer "F.Cu")
-    (at 263.20125 -23.235)
+    (at 263.20125 -20.6355)
     (descr "Footprint for Cherry Clip/Screw in type stabilizers, 2u")
     (property "Sheetfile" "SwitchMatrix.kicad_sch")
@@
   )
   (footprint "marbastlib-mx:STAB_MX_P_7u" (layer "F.Cu")
-    (at 263.20125 -64.895)
+    (at 261.9375 -64.29375)
     (descr "Footprint for Cherry Clip/Screw in type stabilizers, 7u")
     (property "Sheetfile" "SwitchMatrix.kicad_sch")
@@
   )
   (footprint "marbastlib-mx:STAB_MX_2u" (layer "F.Cu")
-    (at 263.20125 -44.065)
+    (at 263.20125 -42.8625)
     (descr "Footprint for Cherry Clip/Screw in type stabilizers, 2u")
     (property "Sheetfile" "SwitchMatrix.kicad_sch")
@@
       (effects (font (size 1 1) (thickness 0.15)))
     )
-    (fp_text value "ISO Enter" (at 0 8.128) (layer "F.Fab")
+    (fp_text value "ISO Enter" (at 0 10.7275) (layer "F.Fab")
       (effects (font (size 1 1) (thickness 0.15)))
     )
@@
       (net 11 "Net-(D4-Pad2)") (pinfunction "2") (pintype "passive"))
   )
+  (footprint "marbastlib-mx:STAB_MX_2u" (layer "F.Cu")
+    (at 261.9375 -126.20625)
+    (descr "Footprint for Cherry Clip/Screw in type stabilizers, 2u")
+    (property "Sheetfile" "SwitchMatrix.kicad_sch")
+    (property "Sheetname" "Switch Matrix")
+    (attr through_hole exclude_from_pos_files)
+    (fp_text reference "S8" (at 0 0) (layer "F.SilkS") hide
+      (effects (font (size 1 1) (thickness 0.15)))
+    )
+    (fp_text value "Enter" (at -1.26375 8.128) (layer "F.Fab")
+      (effects (font (size 1 1) (thickness 0.15)))
+    )
+    (fp_line (start -19.05 -9.525) (end 19.05 -9.525) (layer "Dwgs.User") (width 0.12))
+    (fp_line (start -19.05 -9.525) (end -19.05 9.525) (layer "Dwgs.User") (width 0.12))
+    (fp_line (start 5 7) (end 7 7) (layer "Dwgs.User") (width 0.12))
+    (fp_line (start -19.05 9.525) (end 19.05 9.525) (layer "Dwgs.User") (width 0.12))
+    (fp_line (start 7 7) (end 7 5) (layer "Dwgs.User") (width 0.12))
+    (fp_line (start 5 -7) (end 7 -7) (layer "Dwgs.User") (width 0.12))
+    (fp_line (start -7 7) (end -7 5) (layer "Dwgs.User") (width 0.12))
+    (fp_line (start 19.05 -9.525) (end 19.05 9.525) (layer "Dwgs.User") (width 0.12))
+    (fp_line (start 7 -7) (end 7 -5) (layer "Dwgs.User") (width 0.12))
+    (fp_line (start -5 7) (end -7 7) (layer "Dwgs.User") (width 0.12))
+    (fp_line (start -7 -5) (end -7 -7) (layer "Dwgs.User") (width 0.12))
+    (fp_line (start -7 -7) (end -5 -7) (layer "Dwgs.User") (width 0.12))
+    (fp_line (start 9.03125 -5.999999) (end 14.780039 -5.999999) (layer "Eco2.User") (width 0.05))
+    (fp_line (start -8.53125 -5.499999) (end -8.53125 7.500001) (layer "Eco2.User") (width 0.05))
+    (fp_line (start -14.78125 -5.999999) (end -9.03125 -5.999999) (layer "Eco2.User") (width 0.05))
+    (fp_line (start 15.280039 -5.499999) (end 15.28125 7.500001) (layer "Eco2.User") (width 0.05))
+    (fp_line (start -14.78125 8.000001) (end -9.03125 8.000001) (layer "Eco2.User") (width 0.05))
+    (fp_line (start -15.28125 -5.499999) (end -15.28125 7.500001) (layer "Eco2.User") (width 0.05))
+    (fp_line (start 8.53125 -5.499999) (end 8.53125 7.500001) (layer "Eco2.User") (width 0.05))
+    (fp_line (start 9.03125 8.000001) (end 14.78125 8.000001) (layer "Eco2.User") (width 0.05))
+    (fp_arc (start 15.28125 7.500001) (mid 15.134803 7.853554) (end 14.78125 8.000001) (layer "Eco2.User") (width 0.05))
+    (fp_arc (start -9.03125 -5.999999) (mid -8.677697 -5.853552) (end -8.53125 -5.499999) (layer "Eco2.User") (width 0.05))
+    (fp_arc (start -8.53125 7.500001) (mid -8.677697 7.853554) (end -9.03125 8.000001) (layer "Eco2.User") (width 0.05))
+    (fp_arc (start -15.28125 -5.499999) (mid -15.134803 -5.853552) (end -14.78125 -5.999999) (layer "Eco2.User") (width 0.05))
+    (fp_arc (start 14.780039 -5.999999) (mid 15.133592 -5.853552) (end 15.280039 -5.499999) (layer "Eco2.User") (width 0.05))
+    (fp_arc (start -14.78125 8.000001) (mid -15.134803 7.853554) (end -15.28125 7.500001) (layer "Eco2.User") (width 0.05))
+    (fp_arc (start 9.03125 8.000001) (mid 8.677697 7.853554) (end 8.53125 7.500001) (layer "Eco2.User") (width 0.05))
+    (fp_arc (start 8.53125 -5.499999) (mid 8.677697 -5.853552) (end 9.03125 -5.999999) (layer "Eco2.User") (width 0.05))
+    (fp_circle (center -11.90625 -6.985) (end -9.90625 -6.985) (layer "B.CrtYd") (width 0.12) (fill none))
+    (fp_circle (center 11.90625 -6.985) (end 13.90625 -6.985) (layer "B.CrtYd") (width 0.12) (fill none))
+    (pad "" np_thru_hole circle (at -11.90625 8.255) (size 3.9878 3.9878) (drill 3.9878) (layers *.Cu *.Mask))
+    (pad "" np_thru_hole circle (at -11.90625 -6.985) (size 3.048 3.048) (drill 3.048) (layers *.Cu *.Mask))
+    (pad "" np_thru_hole circle (at 11.90625 8.255) (size 3.9878 3.9878) (drill 3.9878) (layers *.Cu *.Mask))
+    (pad "" np_thru_hole circle (at 11.90625 -6.985) (size 3.048 3.048) (drill 3.048) (layers *.Cu *.Mask))
+    (group "" (id 0a52733a-540c-4fe7-adb1-f079282d1175)
+      (members
+        00385ef4-e786-46e9-8584-865554a29d9d
+        3c25406c-5cea-4e30-b53b-715ee78a5c86
+        51c5189c-34a2-4949-8f49-334f48d29142
+        77e4ff5b-6bf2-4c6c-b880-35f0d82f6183
+        b1f9957a-ffcf-49d8-9eb1-bcdd6046513c
+        c0155609-52a8-4fb8-9cb4-ac8e845abbdf
+        ce9f5807-d322-404e-986a-66d5af1e0047
+        dbea2d37-cf98-4f99-b7a9-f56ddef69ae9
+      )
+    )
+    (group "" (id 63115d88-b487-4b64-a580-a073153ef03b)
+      (members
+        4419de37-1d08-4061-8c3c-3a498cb4091d
+        48c2672d-dbde-4e69-94a7-4d7a00fd9fdb
+        4fd8911a-83dc-46a1-906a-280d1aa5e504
+        50f473d6-2808-4498-8245-d41cc3bc3e66
+        52829f91-dd7a-4c83-9ee3-f41126f0e530
+        77e4bbc3-f936-4787-8acd-0e3cd805be48
+        8abc9e2d-c3af-4027-a75f-64ea8376a470
+        8f39bdd8-90c6-4ac5-83f0-3782f7834fd8
+      )
+    )
+  )
   (footprint "marbastlib-mx:SW_MX_1u" (layer "F.Cu")

Commit message: Position a couple stabs
Parts:
- removed C1: 100nF, marbastlib-mx:STAB_MX_2u
- moved S8 268.2 mm to (307.2, 138.1)
- moved S1 199.9 mm to (309.4, 100.0)
- moved SW47 4.76 mm to (307.2, 138.1)
Changed lines of the file:
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@@
   )
   (footprint "marbastlib-mx:STAB_MX_2u" (layer "F.Cu")
-    (at 383.38125 -85.725)
+    (at 309.4355 100.0125)
     (descr "Footprint for Cherry Clip/Screw in type stabilizers, 2u")
     (property "Sheetfile" "SwitchMatrix.kicad_sch")
@@
   )
   (footprint "marbastlib-mx:SW_MX_1u" (layer "F.Cu")
-    (at 311.94375 138.1125)
+    (at 307.18125 138.1125)
     (descr "Footprint for Cherry MX style switches")
     (tags "cherry mx switch")
@@
   )
   (footprint "marbastlib-mx:STAB_MX_2u" (layer "F.Cu")
-    (at 261.9375 -126.20625)
+    (at 307.18125 138.1125)
     (descr "Footprint for Cherry Clip/Screw in type stabilizers, 2u")
     (property "Sheetfile" "SwitchMatrix.kicad_sch")
@@
     )
   )
-  (footprint "marbastlib-mx:STAB_MX_2u" (layer "B.Cu")
-    (at 538.77 128.23 180)
-    (descr "Footprint for Cherry Clip/Screw in type stabilizers, 2u")
-    (property "Sheetfile" "rp2040-bakeneko65.kicad_sch")
-    (property "Sheetname" "")
-    (attr through_hole exclude_from_pos_files)
-    (fp_text reference "C1" (at 0 0) (layer "B.SilkS") hide
-      (effects (font (size 1 1) (thickness 0.15)) (justify mirror))
-    )
-    (fp_text value "100nF" (at 0 -8.128) (layer "B.Fab")
-      (effects (font (size 1 1) (thickness 0.15)) (justify mirror))
-    )
-    (fp_line (start -7 5) (end -7 7) (layer "Dwgs.User") (width 0.12))
-    (fp_line (start -19.05 9.525) (end -19.05 -9.525) (layer "Dwgs.User") (width 0.12))
-    (fp_line (start 5 7) (end 7 7) (layer "Dwgs.User") (width 0.12))
-    (fp_line (start -7 -7) (end -7 -5) (layer "Dwgs.User") (width 0.12))
-    (fp_line (start -19.05 9.525) (end 19.05 9.525) (layer "Dwgs.User") (width 0.12))
-    (fp_line (start -19.05 -9.525) (end 19.05 -9.525) (layer "Dwgs.User") (width 0.12))
-    (fp_line (start 5 -7) (end 7 -7) (layer "Dwgs.User") (width 0.12))
-    (fp_line (start -5 -7) (end -7 -7) (layer "Dwgs.User") (width 0.12))
-    (fp_line (start -7 7) (end -5 7) (layer "Dwgs.User") (width 0.12))
-    (fp_line (start 19.05 9.525) (end 19.05 -9.525) (layer "Dwgs.User") (width 0.12))
-    (fp_line (start 7 -7) (end 7 -5) (layer "Dwgs.User") (width 0.12))
-    (fp_line (start 7 7) (end 7 5) (layer "Dwgs.User") (width 0.12))
-    (fp_line (start -14.78125 5.999999) (end -9.03125 5.999999) (layer "Eco2.User") (width 0.05))
-    (fp_line (start 8.53125 5.499999) (end 8.53125 -7.500001) (layer "Eco2.User") (width 0.05))
-    (fp_line (start 15.280039 5.499999) (end 15.28125 -7.500001) (layer "Eco2.User") (width 0.05))
-    (fp_line (start -14.78125 -8.000001) (end -9.03125 -8.000001) (layer "Eco2.User") (width 0.05))
-    (fp_line (start 9.03125 5.999999) (end 14.780039 5.999999) (layer "Eco2.User") (width 0.05))
-    (fp_line (start -8.53125 5.499999) (end -8.53125 -7.500001) (layer "Eco2.User") (width 0.05))
-    (fp_line (start -15.28125 5.499999) (end -15.28125 -7.500001) (layer "Eco2.User") (width 0.05))
-    (fp_line (start 9.03125 -8.000001) (end 14.78125 -8.000001) (layer "Eco2.User") (width 0.05))
-    (fp_arc (start -15.28125 -7.500001) (mid -15.134803 -7.853554) (end -14.78125 -8.000001) (layer "Eco2.User") (width 0.05))
-    (fp_arc (start 9.03125 5.999999) (mid 8.677697 5.853552) (end 8.53125 5.499999) (layer "Eco2.User") (width 0.05))
-    (fp_arc (start 8.53125 -7.500001) (mid 8.677697 -7.853554) (end 9.03125 -8.000001) (layer "Eco2.User") (width 0.05))
-    (fp_arc (start -9.03125 -8.000001) (mid -8.677697 -7.853554) (end -8.53125 -7.500001) (layer "Eco2.User") (width 0.05))
-    (fp_arc (start 15.280039 5.499999) (mid 15.133592 5.853552) (end 14.780039 5.999999) (layer "Eco2.User") (width 0.05))
-    (fp_arc (start -8.53125 5.499999) (mid -8.677697 5.853552) (end -9.03125 5.999999) (layer "Eco2.User") (width 0.05))
-    (fp_arc (start 14.78125 -8.000001) (mid 15.134803 -7.853554) (end 15.28125 -7.500001) (layer "Eco2.User") (width 0.05))
-    (fp_arc (start -14.78125 5.999999) (mid -15.134803 5.853552) (end -15.28125 5.499999) (layer "Eco2.User") (width 0.05))
-    (fp_circle (center 11.90625 6.985) (end 13.90625 6.985) (layer "F.CrtYd") (width 0.12) (fill none))
-    (fp_circle (center -11.90625 6.985) (end -9.90625 6.985) (layer "F.CrtYd") (width 0.12) (fill none))
-    (pad "" np_thru_hole circle (at -11.90625 6.985 180) (size 3.048 3.048) (drill 3.048) (layers *.Cu *.Mask))
-    (pad "" np_thru_hole circle (at 11.90625 6.985 180) (size 3.048 3.048) (drill 3.048) (layers *.Cu *.Mask))
-    (pad "" np_thru_hole circle (at 11.90625 -8.255 180) (size 3.9878 3.9878) (drill 3.9878) (layers *.Cu *.Mask))
-    (pad "" np_thru_hole circle (at -11.90625 -8.255 180) (size 3.9878 3.9878) (drill 3.9878) (layers *.Cu *.Mask))
-    (group "" (id 09d5c3f1-2539-4771-b93e-33bdb31609cd)
-      (members
-        13b1f98c-d55e-48c6-bef6-b9e395a5f0b5
-        3fecada7-45e2-483e-87fe-4039d820fb42
-        89eaadca-0685-4163-b755-c48458b69bae
-        96917a2c-4ed8-450b-9658-2f66b858c219
-        c37e3ed7-3a2b-4c9a-8510-29234309c6fe
-        d5eb3f8a-1a63-4b06-83d1-8ffce1049164
-        dcf097d4-ad13-46da-a41d-34742257271d
-        f70f205a-b9f2-4cfd-8d3e-45640e64b241
-      )
-    )
-    (group "" (id e6d2b558-4ee1-48ab-bd93-ea6742ae060c)
-      (members
-        299d0a4e-3447-4115-b4c1-baa7b9336995
-        2a1dd50c-a273-447a-a2e4-20c4605b2193
-        45794be0-d697-453c-a307-6cb73755ae64
-        8b0228c7-b287-4581-bc24-23ead2660862
-        8f0a1ebd-1b2f-4e36-8445-a82769a49312
-        9c65491e-7a6a-44ab-81ee-a4ac811e14f8
-        c72f59d7-5b9a-4d4c-9b3f-03f3ce26787d
-        f8e379fb-e7dd-4ab6-956c-796d8d041a48
-      )
-    )
-  )
