File: plate/SwitchMatrix.kicad_sch (KiCad schematic)
At the start: 166 parts, among them SW1 1u, SW10 1u, SW11 1u, SW12 1u, SW13 1u, SW14 1u, SW15 1u, SW16 1u, SW17 2u, SW18 1.5u, SW19 1u, SW2 1u, SW20 1u, SW21 1u, SW22 1u, SW23 1u, SW24 1u, SW25 1u, SW26 1u, SW27 1u, SW28 1u, SW29 1u, SW3 1u, SW30 1u, SW31 1.5u, SW32 ISO Enter, SW33 1u, SW34 1.25u, SW35 1.75u, SW36 1u, SW37 1u, SW38 1u, SW39 1u, SW4 1u, SW40 1u, SW41 1u, SW42 1u, SW43 1u, SW44 1u, SW45 1u, SW46 1u, SW47 2.25u, SW48 1u, SW49 1u, SW5 1u, SW50 2.25u, SW51 1.25u, SW52 1u, SW53 1u, SW54 1u, SW55 1u, SW56 1u, SW57 1u, SW58 1u, SW59 1u, SW6 1u, SW60 1u, SW61 1u, SW62 1u, SW63 1.75u, SW64 1u, SW65 1u, SW66 1.5u, SW67 1.25u, SW68 1u, SW69 1.25u, SW7 1u, SW70 1.5u, SW71 1.25u, SW72 3u, SW73 2.25u, SW74 7u, SW75 6.25u, SW76 2u, SW77 3u, SW78 2.75u, SW79 1.25u, SW8 1u, SW80 1.5u, SW81 1.25u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

Commit message: swap to PCM footprints
Parts:
- S17, S76: footprint PCM_marbastlib-mx:STAB_MX_P_2u -> marbastlib-mx:STAB_MX_P_2u
- S32: footprint PCM_marbastlib-mx:STAB_MX_P_ISO -> marbastlib-mx:STAB_MX_P_ISO
- S47, S50, S73: footprint PCM_marbastlib-mx:STAB_MX_P_2.25u -> marbastlib-mx:STAB_MX_P_2.25u
- S72, S77: footprint PCM_marbastlib-mx:STAB_MX_P_3u -> marbastlib-mx:STAB_MX_P_3u
- S74: footprint PCM_marbastlib-mx:STAB_MX_P_7u -> marbastlib-mx:STAB_MX_P_7u
- S75: footprint PCM_marbastlib-mx:STAB_MX_P_6.25u -> marbastlib-mx:STAB_MX_P_6.25u
- S78: footprint PCM_marbastlib-mx:STAB_MX_P_2.75u -> marbastlib-mx:STAB_MX_P_2.75u
- SW1, SW10, SW11, SW12, SW13, SW14, SW15, SW16, SW17, SW19, SW2, SW20, SW21, SW22, SW23, SW24, SW25, SW26, SW27, SW28, SW29, SW3, SW30, SW32, SW33, SW36, SW37, SW38, SW39, SW4, SW40, SW41, SW42, SW43, SW44, SW45, SW46, SW47, SW48, SW49, SW5, SW50, SW52, SW53, SW54, SW55, SW56, SW57, SW58, SW59, SW6, SW60, SW61, SW62, SW64, SW65, SW68, SW7, SW72, SW73, SW74, SW75, SW76, SW77, SW78, SW8, SW82, SW83, SW84, SW9: footprint PCM_marbastlib-mx:SW_MX_1u -> marbastlib-mx:SW_MX_1u
- SW18, SW31, SW66, SW70, SW80: footprint PCM_marbastlib-mx:SW_MX_1.5u -> marbastlib-mx:SW_MX_1.5u
- SW34, SW51, SW67, SW69, SW71, SW79, SW81: footprint PCM_marbastlib-mx:SW_MX_1.25u -> marbastlib-mx:SW_MX_1.25u
- SW35, SW63: footprint PCM_marbastlib-mx:SW_MX_1.75u -> marbastlib-mx:SW_MX_1.75u
