File: pcb/rp2040-bakeneko65.kicad_pcb (KiCad board)
At the start: 2 copper layers, 303.8 x 94.2 mm, 201 parts, among them J1 SM04B-SRSS-TB, J2 SWD, SW1 1u, SW10 1u, SW11 1u, SW12 1u, SW13 1u, SW14 1u, SW15 1u, SW16 1u, SW17 2u, SW18 1.5u, SW19 1u, SW2 1u, SW20 1u, SW21 1u, SW22 1u, SW23 1u, SW24 1u, SW25 1u, SW26 1u, SW27 1u, SW28 1u, SW29 1u, SW3 1u, SW30 1u, SW31 1.5u, SW32 ISO Enter, SW33 1u, SW34 1.25u, SW35 1.75u, SW36 1u, SW37 1u, SW38 1u, SW39 1u, SW4 1u, SW40 1u, SW41 1u, SW42 1u, SW43 1u, SW44 1u, SW45 1u, SW46 1u, SW47 2.25u, SW48 1u, SW49 1u, SW5 1u, SW50 2.25u, SW51 1.25u, SW52 1u, SW53 1u, SW54 1u, SW55 1u, SW56 1u, SW57 1u, SW58 1u, SW59 1u, SW6 1u, SW60 1u, SW61 1u, SW62 1u, SW63 1.75u, SW64 1u, SW65 1u, SW66 1.5u, SW67 1.25u, SW68 1u, SW69 1.25u, SW7 1u, SW70 1.5u, SW71 1.25u, SW72 3u, SW73 2.25u, SW74 7u, SW75 6.25u, SW76 2u, SW77 3u, SW78 2.75u, SW79 1.25u, SW8 1u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

Commit message: fix ANSI enter
Parts:
- moved D47 12.3 mm to (331.4, 135.8)
- moved S47 11.9 mm to (323.9, 131.0)
- moved SW48 11.9 mm to (312.0, 131.0)
- moved SW47 11.7 mm to (323.7, 131.0)
- moved D31 0.95 mm to (339.1, 116.7)
Routing:
- net Net-(D47-A): track 38.6 -> 24.6 mm
- net Net-(D31-A): track 38.0 -> 45.1 mm, vias 2 -> 1
- net ROW2: track 333.6 -> 334.9 mm
- net COL15: track 340.7 -> 341.3 mm
- net GND: vias 181 -> 180

Commit message: fix LED capacitor (and update footprints)
and add a missing trace to D47
Parts:
- moved C18 0.76 mm to (71.2, 135.6), turned to 90 degrees
Connections:
- C18 pad 1: +5V -> GND
- C18 pad 2: Net-(LED1-VDD) -> +5V
- LED1 pad 1: Net-(LED1-VDD) -> +5V
Routing:
- net Net-(D47-A): track 24.6 -> 34.8 mm, vias 2 -> 4
- net +5V: track 90.1 -> 93.5 mm
- net Net-(LED1-VDD): track 2.43 -> 0.00 mm
- net GND: track 50.3 -> 51.4 mm
