File: pcb/rp2040-bakeneko65.kicad_sch (KiCad schematic)
At the start: 33 parts, among them J1 SM04B-SRSS-TB, J2 SWD, SW85 SW_Push, U1 RP2040, U2 W25Q128JVS, U3 XC6206PxxxMR, U4 SRV05, Y1 12MHz

Commit message: fix LED capacitor (and update footprints)
and add a missing trace to D47
Connections:
- net +5V: now also C18.2, LED1.1 (VDD); no longer C18.1
- net GND: now also C18.1
Other:
- moved on the sheet: C18, LED1
Changed lines of the file:
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@@
   (junction (at 192.405 31.115) (diameter 0) (color 0 0 0 0)
   )
+  (junction (at 269.24 17.78) (diameter 0) (color 0 0 0 0)
+  )
   (junction (at 259.08 48.26) (diameter 0) (color 0 0 0 0)
   )
@@
   (junction (at 224.79 55.88) (diameter 0) (color 0 0 0 0)
   )
-  (no_connect (at 262.89 24.765))
+  (no_connect (at 262.89 25.4))
   (no_connect (at 97.79 82.55))
   (no_connect (at 97.79 77.47))
@@
     (stroke (width 0) (type default))
   )
+  (wire (pts (xy 269.24 22.86) (xy 269.24 24.13))
+    (stroke (width 0) (type default))
+  )
   (wire (pts (xy 123.825 69.215) (xy 121.285 69.215))
     (stroke (width 0) (type default))
@@
     (stroke (width 0) (type default))
   )
+  (wire (pts (xy 255.27 17.78) (xy 269.24 17.78))
+    (stroke (width 0) (type default))
+  )
   (wire (pts (xy 224.79 55.88) (xy 236.22 55.88))
     (stroke (width 0) (type default))
@@
     (stroke (width 0) (type default))
   )
-  (wire (pts (xy 245.11 17.145) (xy 247.65 17.145))
-    (stroke (width 0) (type default))
-  )
   (wire (pts (xy 123.19 30.48) (xy 124.46 30.48))
     (stroke (width 0) (type default))
@@
     (stroke (width 0) (type default))
   )
-  (wire (pts (xy 252.73 17.145) (xy 255.27 17.145))
-    (stroke (width 0) (type default))
-  )
   (wire (pts (xy 217.17 45.72) (xy 217.17 48.26))
     (stroke (width 0) (type default))
@@
   )
   (wire (pts (xy 247.65 48.26) (xy 259.08 48.26))
+    (stroke (width 0) (type default))
+  )
+  (wire (pts (xy 269.24 16.51) (xy 269.24 17.78))
     (stroke (width 0) (type default))
   )
@@
     )
   )
-  (global_label "LED" (shape input) (at 247.65 24.765 180) (fields_autoplaced)
+  (global_label "LED" (shape input) (at 247.65 25.4 180) (fields_autoplaced)
     (effects (font (size 1.27 1.27)) (justify right))
-    (property "Intersheetrefs" "${INTERSHEET_REFS}" (at 241.7898 24.6856 0)
+    (property "Intersheetrefs" "${INTERSHEET_REFS}" (at 241.7898 25.3206 0)
       (effects (font (size 1.27 1.27)) (justify right) hide)
     )
@@
         (path "/6136f036-b0e3-42a2-8ab6-1b828fccf946"
           (reference "SW85") (unit 1)
+        )
+      )
+    )
+  )
+  (symbol (lib_name "+5V_1") (lib_id "power:+5V") (at 269.24 16.51 0) (unit 1)
+    (in_bom yes) (on_board yes) (dnp no)
+    (property "Reference" "#PWR067" (at 269.24 20.32 0)
+      (effects (font (size 1.27 1.27)) hide)
+    )
+    (property "Value" "+5V" (at 265.43 15.24 0)
+      (effects (font (size 1.27 1.27)))
+    )
+    (property "Footprint" "" (at 269.24 16.51 0)
+      (effects (font (size 1.27 1.27)) hide)
+    )
+    (property "Datasheet" "" (at 269.24 16.51 0)
+      (effects (font (size 1.27 1.27)) hide)
+    )
+    (pin "1")
+    (instances
+      (project "rp2040-bakeneko65"
+        (path "/6136f036-b0e3-42a2-8ab6-1b828fccf946"
+          (reference "#PWR067") (unit 1)
         )
       )
@@
     )
   )
-  (symbol (lib_id "power:GND") (at 255.27 32.385 0) (unit 1)
-    (in_bom yes) (on_board yes) (dnp no)
-    (property "Reference" "#PWR0106" (at 255.27 38.735 0)
-      (effects (font (size 1.27 1.27)) hide)
-    )
-    (property "Value" "GND" (at 257.81 32.385 0)
-      (effects (font (size 1.27 1.27)))
-    )
-    (property "Footprint" "" (at 255.27 32.385 0)
-      (effects (font (size 1.27 1.27)) hide)
-    )
-    (property "Datasheet" "" (at 255.27 32.385 0)
+  (symbol (lib_id "power:GND") (at 255.27 33.02 0) (unit 1)
+    (in_bom yes) (on_board yes) (dnp no)
+    (property "Reference" "#PWR0106" (at 255.27 39.37 0)
+      (effects (font (size 1.27 1.27)) hide)
+    )
+    (property "Value" "GND" (at 257.81 33.02 0)
+      (effects (font (size 1.27 1.27)))
+    )
+    (property "Footprint" "" (at 255.27 33.02 0)
+      (effects (font (size 1.27 1.27)) hide)
+    )
+    (property "Datasheet" "" (at 255.27 33.02 0)
       (effects (font (size 1.27 1.27)) hide)
     )
@@
     )
   )
-  (symbol (lib_id "Device:C_Small") (at 250.19 17.145 90) (unit 1)
-    (in_bom yes) (on_board yes) (dnp no)
-    (property "Reference" "C18" (at 248.285 13.97 90)
-      (effects (font (size 1.27 1.27)))
-    )
-    (property "Value" "100nF" (at 254.635 13.97 90)
-      (effects (font (size 1.27 1.27)))
-    )
-    (property "Footprint" "Capacitor_SMD:C_0402_1005Metric" (at 250.19 17.145 0)
-      (effects (font (size 1.27 1.27)) hide)
-    )
-    (property "Datasheet" "~" (at 250.19 17.145 0)
+  (symbol (lib_id "Device:C_Small") (at 269.24 20.32 180) (unit 1)
+    (in_bom yes) (on_board yes) (dnp no)
+    (property "Reference" "C18" (at 273.05 17.78 0)
+      (effects (font (size 1.27 1.27)))
+    )
+    (property "Value" "100nF" (at 274.32 20.32 0)
+      (effects (font (size 1.27 1.27)))
+    )
+    (property "Footprint" "Capacitor_SMD:C_0402_1005Metric" (at 269.24 20.32 0)
+      (effects (font (size 1.27 1.27)) hide)
+    )
+    (property "Datasheet" "~" (at 269.24 20.32 0)
       (effects (font (size 1.27 1.27)) hide)
     )
@@
         (path "/6136f036-b0e3-42a2-8ab6-1b828fccf946"
           (reference "#PWR066") (unit 1)
+        )
+      )
+    )
+  )
+  (symbol (lib_name "GND_3") (lib_id "power:GND") (at 269.24 24.13 0) (unit 1)
+    (in_bom yes) (on_board yes) (dnp no)
+    (property "Reference" "#PWR068" (at 269.24 30.48 0)
+      (effects (font (size 1.27 1.27)) hide)
+    )
+    (property "Value" "GND" (at 273.05 25.4 0)
+      (effects (font (size 1.27 1.27)))
+    )
+    (property "Footprint" "" (at 269.24 24.13 0)
+      (effects (font (size 1.27 1.27)) hide)
+    )
+    (property "Datasheet" "" (at 269.24 24.13 0)
+      (effects (font (size 1.27 1.27)) hide)
+    )
+    (pin "1")
+    (instances
+      (project "rp2040-bakeneko65"
+        (path "/6136f036-b0e3-42a2-8ab6-1b828fccf946"
+          (reference "#PWR068") (unit 1)
         )
       )
@@
     )
   )
-  (symbol (lib_id "power:+5V") (at 245.11 17.145 0) (unit 1)
-    (in_bom yes) (on_board yes) (dnp no)
-    (property "Reference" "#PWR0124" (at 245.11 20.955 0)
-      (effects (font (size 1.27 1.27)) hide)
-    )
-    (property "Value" "+5V" (at 241.935 17.145 0)
-      (effects (font (size 1.27 1.27)))
-    )
-    (property "Footprint" "" (at 245.11 17.145 0)
-      (effects (font (size 1.27 1.27)) hide)
-    )
-    (property "Datasheet" "" (at 245.11 17.145 0)
-      (effects (font (size 1.27 1.27)) hide)
-    )
-    (pin "1")
-    (instances
-      (project "rp2040-bakeneko65"
-        (path "/6136f036-b0e3-42a2-8ab6-1b828fccf946"
-          (reference "#PWR0124") (unit 1)
-        )
-      )
-    )
-  )
-  (symbol (lib_id "marbastlib-mx:MX_SK6812MINI-E") (at 255.27 24.765 0) (unit 1)
-    (in_bom yes) (on_board yes) (dnp no)
-    (property "Reference" "LED1" (at 264.16 27.94 0)
-      (effects (font (size 1.27 1.27)))
-    )
-    (property "Value" "SK6812 Mini-E" (at 269.24 30.48 0)
-      (effects (font (size 1.27 1.27)))
-    )
-    (property "Footprint" "PCM_marbastlib-mx:LED_MX_6028R" (at 255.27 24.765 0)
-      (effects (font (size 1.27 1.27)) hide)
-    )
-    (property "Datasheet" "" (at 255.27 24.765 0)
-      (effects (font (size 1.27 1.27)) hide)
-    )
+  (symbol (lib_id "marbastlib-mx:MX_SK6812MINI-E") (at 255.27 25.4 0) (unit 1)
+    (in_bom yes) (on_board yes) (dnp no)
+    (property "Reference" "LED1" (at 264.16 28.575 0)
+      (effects (font (size 1.27 1.27)))
+    )
+    (property "Value" "SK6812 Mini-E" (at 269.24 31.115 0)
+      (effects (font (size 1.27 1.27)))
+    )
+    (property "Footprint" "PCM_marbastlib-mx:LED_MX_6028R" (at 255.27 25.4 0)
+      (effects (font (size 1.27 1.27)) hide)
+    )
+    (property "Datasheet" "" (at 255.27 25.4 0)
+      (effects (font (size 1.27 1.27)) hide)
+    )
